File: designs/radPi/motors.sch (KiCad schematic (older format))
At the start: 13 parts, among them K1 LEMO2, P5 PUMP_OUT, Q1 BC556, SW1 G6DN_Relay

Commit message: restructured radishes for nubby branch
Parts:
- C1, C2: symbol CP -> radPi-rescue:CP
- C3: symbol C -> radPi-rescue:C
- D1, D3: symbol D -> radPi-rescue:D
- D2: symbol LED -> radPi-rescue:LED
- K1: symbol LEMO2-RESCUE-radPi -> radPi-rescue:LEMO2-RESCUE-radPi
- L1: symbol L -> radPi-rescue:L
- P5: symbol CONN_01X02 -> radPi-rescue:CONN_01X02
- Q1: symbol BC556 -> radPi-rescue:BC556
- R1, R2: symbol R -> radPi-rescue:R
- SW1: symbol G6DN_Relay -> relays:G6DN_Relay
Changed lines of the file:
@@
-EESchema Schematic File Version 2
-LIBS:radPi-rescue
-LIBS:power
-LIBS:device
-LIBS:transistors
-LIBS:conn
-LIBS:linear
-LIBS:regul
-LIBS:74xx
-LIBS:cmos4000
-LIBS:adc-dac
-LIBS:memory
-LIBS:xilinx
-LIBS:microcontrollers
-LIBS:dsp
-LIBS:microchip
-LIBS:analog_switches
-LIBS:motorola
-LIBS:texas
-LIBS:intel
-LIBS:audio
-LIBS:interface
-LIBS:digital-audio
-LIBS:philips
-LIBS:display
-LIBS:cypress
-LIBS:siliconi
-LIBS:opto
-LIBS:atmel
-LIBS:contrib
-LIBS:valves
-LIBS:devs
-LIBS:relays
+EESchema Schematic File Version 4
 LIBS:radPi-cache
-EELAYER 25 0
+EELAYER 26 0
 EELAYER END
 $Descr A4 11693 8268
@@
 $EndDescr
 $Comp
-L LEMO2-RESCUE-radPi K?
+L radPi-rescue:LEMO2-RESCUE-radPi K?
 U 1 1 59B32C2E
 P 3950 1950
@@
 $EndComp
 $Comp
-L GND #PWR011
+L power:GND #PWR011
 U 1 1 59B32CBE
 P 3750 2200
@@
 $EndComp
 $Comp
-L +12V #PWR012
+L power:+12V #PWR012
 U 1 1 59B32CE4
 P 4200 2250
@@
 $EndComp
 $Comp
-L G6DN_Relay SW1
+L relays:G6DN_Relay SW1
 U 1 1 59B5F092
 P 3250 3050
@@
 $EndComp
 $Comp
-L D D1
+L radPi-rescue:D D1
 U 1 1 59B5F17D
 P 2200 3050
@@
 PUMP_IN
 $Comp
-L C C3
+L radPi-rescue:C C3
 U 1 1 59B60A7A
 P 4500 3450
@@
 $EndComp
 $Comp
-L CP C2
+L radPi-rescue:CP C2
 U 1 1 59B60AE8
 P 4250 2750
@@
 $EndComp
 $Comp
-L CONN_01X02 P5
+L radPi-rescue:CONN_01X02 P5
 U 1 1 59B60C39
 P 5150 3450
@@
 $EndComp
 $Comp
-L GND #PWR013
+L power:GND #PWR013
 U 1 1 59B610C8
 P 2200 3650
@@
 $EndComp
 $Comp
-L LED D2
+L radPi-rescue:LED D2
 U 1 1 59B616E3
 P 4250 4000
@@
 $EndComp
 $Comp
-L R R2
+L radPi-rescue:R R2
 U 1 1 59B618AA
 P 4250 3550
@@
 $EndComp
 $Comp
-L GNDD #PWR014
+L power:GNDD #PWR014
 U 1 1 59B62B40
 P 4250 2950
@@
 $EndComp
 $Comp
-L GNDD #PWR015
+L power:GNDD #PWR015
 U 1 1 59B62B9D
 P 3350 4150
@@
 $EndComp
 $Comp
-L GND #PWR016
+L power:GND #PWR016
 U 1 1 59B62C20
 P 3050 4150
@@
 $EndComp
 $Comp
-L L L1
+L radPi-rescue:L L1
 U 1 1 59B62C45
 P 3200 4100
@@
 $EndComp
 $Comp
-L R R1
+L radPi-rescue:R R1
 U 1 1 59B5F2DD
 P 1350 3300
@@
 $EndComp
 $Comp
-L BC556 Q1
+L radPi-rescue:BC556 Q1
 U 1 1 59B65C2E
 P 1700 3300
@@
 $EndComp
 $Comp
-L D D3
+L radPi-rescue:D D3
 U 1 1 59B65D7A
 P 4750 3450
@@
 	4250 2950 4250 2900
 $Comp
-L GNDD #PWR017
+L power:GNDD #PWR017
 U 1 1 59B6663B
 P 4250 4250
@@
 $EndComp
 $Comp
-L CP C1
+L radPi-rescue:CP C1
 U 1 1 59B71339
 P 2450 3050
