File: designs/radPi/radPi.sch (KiCad schematic (older format))
At the start: 1 part, among them U1 RaspberryPi3_ModB

Commit message: restructured radishes for nubby branch
Parts:
- U1: symbol RaspberryPi3_ModB-RESCUE-radPi -> radPi-rescue:RaspberryPi3_ModB-RESCUE-radPi
Changed lines of the file:
@@
-EESchema Schematic File Version 2
-LIBS:radPi-rescue
-LIBS:power
-LIBS:device
-LIBS:transistors
-LIBS:conn
-LIBS:linear
-LIBS:regul
-LIBS:74xx
-LIBS:cmos4000
-LIBS:adc-dac
-LIBS:memory
-LIBS:xilinx
-LIBS:microcontrollers
-LIBS:dsp
-LIBS:microchip
-LIBS:analog_switches
-LIBS:motorola
-LIBS:texas
-LIBS:intel
-LIBS:audio
-LIBS:interface
-LIBS:digital-audio
-LIBS:philips
-LIBS:display
-LIBS:cypress
-LIBS:siliconi
-LIBS:opto
-LIBS:atmel
-LIBS:contrib
-LIBS:valves
-LIBS:devs
-LIBS:relays
+EESchema Schematic File Version 4
 LIBS:radPi-cache
-EELAYER 25 0
+EELAYER 26 0
 EELAYER END
 $Descr A4 11693 8268
@@
 $EndDescr
 $Comp
-L RaspberryPi3_ModB-RESCUE-radPi U1
+L radPi-rescue:RaspberryPi3_ModB-RESCUE-radPi U1
 U 1 1 59B1EDFB
 P 2800 3600
@@
 $EndSheet
 $Comp
-L +5V #PWR01
+L power:+5V #PWR01
 U 1 1 59B1FB01
 P 3150 1300
@@
 $EndComp
 $Comp
-L +5V #PWR02
+L power:+5V #PWR02
 U 1 1 59B1FC65
 P 4200 1700
@@
 $EndComp
 $Comp
-L +3.3V #PWR03
+L radPi-rescue:+3.3V #PWR03
 U 1 1 59B27B65
 P 2450 1300
@@
 $EndSheet
 $Comp
-L GND #PWR04
+L power:GND #PWR04
 U 1 1 59B66C8E
 P 2350 5900
@@
 	2350 5900 2350 5800
 Wire Wire Line
-	2350 5800 2750 5800
+	2350 5800 2450 5800
 Connection ~ 2450 5800
 Connection ~ 2550 5800
 Connection ~ 2650 5800
 $Comp
-L PWR_FLAG #FLG05
+L power:PWR_FLAG #FLG05
 U 1 1 59D95B93
 P 950 1000
@@
 $EndComp
 $Comp
-L +3.3V #PWR06
+L radPi-rescue:+3.3V #PWR06
 U 1 1 59D95C61
 P 950 900
@@
 Wire Wire Line
 	950  900  950  1000
+Wire Wire Line
+	2450 5800 2550 5800
+Wire Wire Line
+	2550 5800 2650 5800
+Wire Wire Line
+	2650 5800 2750 5800
 $EndSCHEMATC
