File: designs/radPi/sensors.sch (KiCad schematic (older format))
At the start: 8 parts, among them P1 CONN_01X04, P2 CONN_01X04, P3 CONN_01X04, P4 CONN_01X04, U2 ADS1115, U3 ADS1115, U4 ADS1115, U5 ADS1115

Commit message: restructured radishes for nubby branch
Parts:
- P1, P2, P3, P4: symbol CONN_01X04 -> radPi-rescue:CONN_01X04
- U2, U3, U4, U5: symbol ADS1115 -> devs:ADS1115
Changed lines of the file:
@@
-EESchema Schematic File Version 2
-LIBS:radPi-rescue
-LIBS:power
-LIBS:device
-LIBS:transistors
-LIBS:conn
-LIBS:linear
-LIBS:regul
-LIBS:74xx
-LIBS:cmos4000
-LIBS:adc-dac
-LIBS:memory
-LIBS:xilinx
-LIBS:microcontrollers
-LIBS:dsp
-LIBS:microchip
-LIBS:analog_switches
-LIBS:motorola
-LIBS:texas
-LIBS:intel
-LIBS:audio
-LIBS:interface
-LIBS:digital-audio
-LIBS:philips
-LIBS:display
-LIBS:cypress
-LIBS:siliconi
-LIBS:opto
-LIBS:atmel
-LIBS:contrib
-LIBS:valves
-LIBS:devs
-LIBS:relays
+EESchema Schematic File Version 4
 LIBS:radPi-cache
-EELAYER 25 0
+EELAYER 26 0
 EELAYER END
 $Descr A4 11693 8268
@@
 $EndDescr
 $Comp
-L ADS1115 U3
+L devs:ADS1115 U3
 U 1 1 59B29154
 P 6250 1950
@@
 $EndComp
 $Comp
-L ADS1115 U4
+L devs:ADS1115 U4
 U 1 1 59B29192
 P 6250 3250
@@
 $EndComp
 $Comp
-L ADS1115 U5
+L devs:ADS1115 U5
 U 1 1 59B291B4
 P 6250 4550
@@
 $EndComp
 $Comp
-L ADS1115 U2
+L devs:ADS1115 U2
 U 1 1 59B29207
 P 6200 5850
@@
 Connection ~ 4600 4100
 $Comp
-L GND #PWR07
+L power:GND #PWR07
 U 1 1 59B29CD3
 P 5150 1650
@@
 $EndComp
 $Comp
-L GND #PWR08
+L power:GND #PWR08
 U 1 1 59B29D2D
 P 5200 2950
@@
 $EndComp
 $Comp
-L GND #PWR09
+L power:GND #PWR09
 U 1 1 59B29D44
 P 5250 4250
@@
 $EndComp
 $Comp
-L GND #PWR010
+L power:GND #PWR010
 U 1 1 59B29DB3
 P 5250 5550
@@
 	5800 3300 5750 3300
 $Comp
-L CONN_01X04 P2
+L radPi-rescue:CONN_01X04 P2
 U 1 1 59B2AE3D
 P 5100 3550
@@
 	5750 2000 5800 2000
 $Comp
-L CONN_01X04 P1
+L radPi-rescue:CONN_01X04 P1
 U 1 1 59B2B108
 P 5100 2250
@@
 $EndComp
 $Comp
-L CONN_01X04 P3
+L radPi-rescue:CONN_01X04 P3
 U 1 1 59B2B15A
 P 5100 4850
@@
 $EndComp
 $Comp
-L CONN_01X04 P4
+L radPi-rescue:CONN_01X04 P4
 U 1 1 59B2B315
 P 5100 6150
