File: hardware/sensor-interface/sableye.sch (KiCad schematic (older format))
At the start: 9 parts, among them J1 Conn_PiWR-Pi2C-PiLERTs, J2 Conn_A0x48-9, J3 Conn_A0x4A-B, J4 Conn_Bonus-I2C, U1 ADS1115, U2 ADS1115, U3 ADS1115, U4 ADS1115

Commit message: Started re-re-design i2c interface board for fitting more ADCs onboard; needs some more work to accommodate other sensors
Parts:
- removed J4: Conn_Bonus-I2C, Connector_Phoenix_MC_HighVoltage:PhoenixContact_MC_1,5_8-G-5.08_1x08_P5.08mm_Horizontal, symbol Connector:Conn_01x08_Female
- added C2, C3, C4, C5: 1uF, Capacitor_SMD:C_0805_2012Metric_Pad1.15x1.40mm_HandSolder, symbol Device:C
- added FB1, FB2: MMZ2012Y152B, Inductor_SMD:L_0805_2012Metric_Pad1.15x1.40mm_HandSolder, symbol Device:Ferrite_Bead
- added R1, R2, R3, R4, R5, R6: 10k, Resistor_SMD:R_0805_2012Metric_Pad1.15x1.40mm_HandSolder, symbol Device:R
- C1: value C_PWR (optional) -> 1uF
- U1, U2, U3, U4: footprint Connector_PinHeader_2.54mm:PinHeader_1x10_P2.54mm_Vertical -> Radishes:VSSOP-10_2.4x2.1mm_P0.5mm
Connections:
- wire segments 100 -> 137
Other:
- note added: "NOTES:\n * Add ADC address labels to silkscreen.\n * Place protection capacitors physically close to ADS1115s.\n * Current ferrite beads only spec'd for <500mA."
- note added: "TODO:\n *Layout\n * Needs to accommodate soil sensor, temp/humidity sensors."
- moved on the sheet: C1
